Commit message: drafted tether heading indicator block

File: objects/robot_blue.urdf (robot description, URDF)
Before this commit: robot disk, 5 links, 4 joints
Links:
- added link tether_block, mass 0.01; collision box size=0.02 0.01 0.01; visual box size=0.02 0.01 0.01
Joints:
- added joint tether_block_to_base: type continuous, parent base_link, child tether_block, origin xyz=$0.1 0 $0.005 rpy=0 0 0, axis 0 0 1, limit effort=0 velocity=1000

Commit message: fixed get_tether_heading to rely on properties of the agent and its tether rather than the position of other agents

File: objects/robot_blue.urdf (robot description, URDF)
Before this commit: robot disk, 6 links, 5 joints
Links:
- removed link tether_block
Joints:
- removed joint tether_block_to_base
